Commit message: deployment for repo publishing

File: assets/urdf/NICOL.urdf (robot description, URDF)
Before this commit: robot NICOL, 99 links, 98 joints
Links:
- link base_link: geometry collision box size=0.045 0.1 1.0; visual mesh filename=package://nias_description/meshes/robot_frame/holder_with_s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 scale=0.001 0.001 0.001
- link camera_holder_link: geometry collision box size=0 0 0; visual mesh filename=package://nias_description/meshes/robot_frame/camera_holder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 scale=0.001 0.001 0.001
- link camera_link: geometry collision box size=0 0 0; visual mesh filename=package://nias_description/meshes/camera/Intel_RealSense_De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 scale=0.001 0.001 0.001
- link face_link: geometry collision cylinder length=0.24 radius=0.128; visual mesh filename=package://nias_description/meshes/head/high_res/NICOL_1x3_c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 scale=0.001 0.001 0.001
- link frame_link: geometry collision box size=0 0 0; visual mesh filename=package://nias_description/meshes/robot_frame/robot_frame_c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 scale=0.001 0.001 0.001
- link l_Ibumper: geometry collision mesh filename=package://nias_description/meshes/RH8D/high_res/sensor_refa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 scale=0.001 0.001 0.001; visual mesh filename=package://nias_description/meshes/RH8D/high_res/sensor_refa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 scale=0.001 0.001 0.001
- link l_Imiddle: geometry collision mesh filename=package://nias_description/meshes/RH8D/phalanx_refac.stl scale=0.001 0.001 0.001; visual mesh filename=package://nias_description/meshes/RH8D/phalanx_refac.stl scale=0.001 0.001 0.001
- link l_Iproximal: geometry collision mesh filename=package://nias_description/meshes/RH8D/phalanx_refac.stl scale=0.001 0.001 0.001; visual mesh filename=package://nias_description/meshes/RH8D/phalanx_refac.stl scale=0.001 0.001 0.001
- link l_Itip: geometry collision mesh filename=package://nias_description/meshes/RH8D/high_res/tip_refac.s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 scale=0.001 0.001 0.001; visual mesh filename=package://nias_description/meshes/RH8D/high_res/tip_refac.s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 scale=0.001 0.001 0.001
- link l_Lbumper: geometry collision mesh filename=package://nias_description/meshes/RH8D/high_res/sensor_refa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 scale=0.001 0.001 0.001; visual mesh filename=package://nias_description/meshes/RH8D/high_res/sensor_refa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 scale=0.001 0.001 0.001
- link l_Lmiddle: geometry collision mesh filename=package://nias_description/meshes/RH8D/phalanx_refac.stl scale=0.001 0.001 0.001; visual mesh filename=package://nias_description/meshes/RH8D/phalanx_refac.stl scale=0.001 0.001 0.001
- link l_Lproximal: geometry collision mesh filename=package://nias_description/meshes/RH8D/phalanx_refac.stl scale=0.001 0.001 0.001; visual mesh filename=package://nias_description/meshes/RH8D/phalanx_refac.stl scale=0.001 0.001 0.001
- link l_Ltip: geometry collision mesh filename=package://nias_description/meshes/RH8D/high_res/tip_refac.s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 scale=0.001 0.001 0.001; visual mesh filename=package://nias_description/meshes/RH8D/high_res/tip_refac.s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 scale=0.001 0.001 0.001
- link l_Mbumper: geometry collision mesh filename=package://nias_description/meshes/RH8D/high_res/optoforce_s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 scale=0.001 0.001 0.001; visual mesh filename=package://nias_description/meshes/RH8D/high_res/optoforce_s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 scale=0.001 0.001 0.001
- link l_Mmiddle: geometry collision mesh filename=package://nias_description/meshes/RH8D/phalanx_refac.stl scale=0.001 0.001 0.001; visual mesh filename=package://nias_description/meshes/RH8D/phalanx_refac.stl scale=0.001 0.001 0.001
- link l_Mproximal: geometry collision mesh filename=package://nias_description/meshes/RH8D/phalanx_refac.stl scale=0.001 0.001 0.001; visual mesh filename=package://nias_description/meshes/RH8D/phalanx_refac.stl scale=0.001 0.001 0.001
- link l_Mtip: geometry collision mesh filename=package://nias_description/meshes/RH8D/high_res/optoforce_t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 scale=0.001 0.001 0.001; visual mesh filename=package://nias_description/meshes/RH8D/high_res/optoforce_t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 scale=0.001 0.001 0.001
- link l_Rbumper: geometry collision mesh filename=package://nias_description/meshes/RH8D/high_res/sensor_refa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 scale=0.001 0.001 0.001; visual mesh filename=package://nias_description/meshes/RH8D/high_res/sensor_refa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 scale=0.001 0.001 0.001
- link l_Rmiddle: geometry collision mesh filename=package://nias_description/meshes/RH8D/phalanx_refac.stl scale=0.001 0.001 0.001; visual mesh filename=package://nias_description/meshes/RH8D/phalanx_refac.stl scale=0.001 0.001 0.001
- link l_Rproximal: geometry collision mesh filename=package://nias_description/meshes/RH8D/phalanx_refac.stl scale=0.001 0.001 0.001; visual mesh filename=package://nias_description/meshes/RH8D/phalanx_refac.stl scale=0.001 0.001 0.001
- link l_Rtip: geometry collision mesh filename=package://nias_description/meshes/RH8D/high_res/tip_refac.s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 scale=0.001 0.001 0.001; visual mesh filename=package://nias_description/meshes/RH8D/high_res/tip_refac.s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 scale=0.001 0.001 0.001
- link l_Tbumper: geometry collision mesh filename=package://nias_description/meshes/RH8D/high_res/sensor_refa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 scale=0.001 0.001 0.001; visual mesh filename=package://nias_description/meshes/RH8D/high_res/sensor_refa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 scale=0.001 0.001 0.001
- link l_Tmiddle: geometry collision mesh filename=package://nias_description/meshes/RH8D/thumb_phalanx_refac.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 scale=0.001 0.001 0.001; visual mesh filename=package://nias_description/meshes/RH8D/thumb_phalanx_refac.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 scale=0.001 0.001 0.001
- link l_Tproximal: geometry collision mesh filename=package://nias_description/meshes/RH8D/thumb_phalanx_col.stl scale=0.001 0.001 0.001; visual mesh filename=package://nias_description/meshes/RH8D/thumb_phalanx_refac.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 scale=0.001 0.001 0.001
- link l_Ttip: geometry collision mesh filename=package://nias_description/meshes/RH8D/high_res/tip_refac.s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 scale=0.001 0.001 0.001; visual mesh filename=package://nias_description/meshes/RH8D/high_res/tip_refac.s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 scale=0.001 0.001 0.001
- link l_forearm: geometry collision mesh filename=package://nias_description/meshes/RH8D/forearm_refac.stl scale=0.001 0.001 0.001; visual mesh filename=package://nias_description/meshes/RH8D/forearm_refac.stl scale=0.001 0.001 0.001
- link l_link1: geometry collision box size=0.055 0.055 0.13; visual mesh filename=package://nias_description/meshes/open_manipulator/link_1_r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 scale=0.001 0.001 0.001
- link l_link2: geometry collision box size=0.055 0.1325 0.055; visual mesh filename=package://nias_description/meshes/open_manipulator/link_2_r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 scale=0.001 0.001 0.001
- link l_link3: geometry collision mesh filename=package://nias_description/meshes/open_manipulator/link_3_r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 scale=0.001 0.001 0.001; visual mesh filename=package://nias_description/meshes/open_manipulator/link_3_r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 scale=0.001 0.001 0.001
- link l_link4: geometry collision mesh filename=package://nias_description/meshes/open_manipulator/link_4_r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 scale=0.001 0.001 0.001; visual mesh filename=package://nias_description/meshes/open_manipulator/link_4_r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 scale=0.001 0.001 0.001
- link l_link5: geometry collision box size=0.047 0.08 0.05; visual mesh filename=package://nias_description/meshes/open_manipulator/link_5_r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 scale=0.001 0.001 0.001
- link l_link6: geometry collision mesh filename=package://nias_description/meshes/open_manipulator/link_6_r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 scale=0.001 0.001 0.001; visual mesh filename=package://nias_description/meshes/open_manipulator/link_6_r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 scale=0.001 0.001 0.001
- link l_palm: geometry collision mesh filename=package://nias_description/meshes/RH8D/high_res/left_palm_r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 scale=0.001 0.001 0.001; visual mesh filename=package://nias_description/meshes/RH8D/high_res/left_palm_r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 scale=0.001 0.001 0.001
- link l_palm_axis: geometry collision mesh filename=package://nias_description/meshes/RH8D/palm_axis_refac.stl scale=0.001 0.001 0.001; visual mesh filename=package://nias_description/meshes/RH8D/palm_axis_refac.stl scale=0.001 0.001 0.001
- link l_thumb_base: geometry collision box size=0 0 0; visual mesh filename=package://nias_description/meshes/RH8D/thumb_base_refac.stl scale=0.001 0.001 0.001
- link left_eye_link: geometry collision box size=0 0 0; visual mesh filename=package://nias_description/meshes/head/BF10M10526S132C_cent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 scale=0.001 0.001 0.001
- link neck_link: geometry collision cylinder length=0.13 radius=0.038; visual mesh filename=package://nias_description/meshes/head/cplt_neck_asmbly.stl scale=0.001 0.001 0.001
- link occiput_link: geometry collision box size=0 0 0; visual mesh filename=package://nias_description/meshes/head/occiput_1x3_centered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 scale=0.001 0.001 0.001
- link plate_link: geometry collision box size=1.0 2.0 0.02; visual mesh filename=package://nias_description/meshes/robot_frame/plate_centere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 scale=0.001 0.001 0.001
- link r_Ibumper: geometry collision mesh filename=package://nias_description/meshes/RH8D/high_res/sensor_refa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 scale=0.001 0.001 0.001; visual mesh filename=package://nias_description/meshes/RH8D/high_res/sensor_refa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 scale=0.001 0.001 0.001
- link r_Imiddle: geometry collision mesh filename=package://nias_description/meshes/RH8D/phalanx_refac.stl scale=0.001 0.001 0.001; visual mesh filename=package://nias_description/meshes/RH8D/phalanx_refac.stl scale=0.001 0.001 0.001
- link r_Iproximal: geometry collision mesh filename=package://nias_description/meshes/RH8D/phalanx_refac.stl scale=0.001 0.001 0.001; visual mesh filename=package://nias_description/meshes/RH8D/phalanx_refac.stl scale=0.001 0.001 0.001
- link r_Itip: geometry collision mesh filename=package://nias_description/meshes/RH8D/high_res/tip_refac.s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 scale=0.001 0.001 0.001; visual mesh filename=package://nias_description/meshes/RH8D/high_res/tip_refac.s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 scale=0.001 0.001 0.001
- link r_Lbumper: geometry collision mesh filename=package://nias_description/meshes/RH8D/high_res/sensor_refa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 scale=0.001 0.001 0.001; visual mesh filename=package://nias_description/meshes/RH8D/high_res/sensor_refa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 scale=0.001 0.001 0.001
- link r_Lmiddle: geometry collision mesh filename=package://nias_description/meshes/RH8D/phalanx_refac.stl scale=0.001 0.001 0.001; visual mesh filename=package://nias_description/meshes/RH8D/phalanx_refac.stl scale=0.001 0.001 0.001
- link r_Lproximal: geometry collision mesh filename=package://nias_description/meshes/RH8D/phalanx_refac.stl scale=0.001 0.001 0.001; visual mesh filename=package://nias_description/meshes/RH8D/phalanx_refac.stl scale=0.001 0.001 0.001
- link r_Ltip: geometry collision mesh filename=package://nias_description/meshes/RH8D/high_res/tip_refac.s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 scale=0.001 0.001 0.001; visual mesh filename=package://nias_description/meshes/RH8D/high_res/tip_refac.s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 scale=0.001 0.001 0.001
- link r_Mbumper: geometry collision mesh filename=package://nias_description/meshes/RH8D/high_res/sensor_refa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 scale=0.001 0.001 0.001; visual mesh filename=package://nias_description/meshes/RH8D/high_res/sensor_refa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 scale=0.001 0.001 0.001
- link r_Mmiddle: geometry collision mesh filename=package://nias_description/meshes/RH8D/phalanx_refac.stl scale=0.001 0.001 0.001; visual mesh filename=package://nias_description/meshes/RH8D/phalanx_refac.stl scale=0.001 0.001 0.001
- link r_Mproximal: geometry collision mesh filename=package://nias_description/meshes/RH8D/phalanx_refac.stl scale=0.001 0.001 0.001; visual mesh filename=package://nias_description/meshes/RH8D/phalanx_refac.stl scale=0.001 0.001 0.001
- link r_Mtip: geometry collision mesh filename=package://nias_description/meshes/RH8D/high_res/tip_refac.s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 scale=0.001 0.001 0.001; visual mesh filename=package://nias_description/meshes/RH8D/high_res/tip_refac.s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 scale=0.001 0.001 0.001
- link r_Rbumper: geometry collision mesh filename=package://nias_description/meshes/RH8D/high_res/sensor_refa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 scale=0.001 0.001 0.001; visual mesh filename=package://nias_description/meshes/RH8D/high_res/sensor_refa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 scale=0.001 0.001 0.001
- link r_Rmiddle: geometry collision mesh filename=package://nias_description/meshes/RH8D/phalanx_refac.stl scale=0.001 0.001 0.001; visual mesh filename=package://nias_description/meshes/RH8D/phalanx_refac.stl scale=0.001 0.001 0.001
- link r_Rproximal: geometry collision mesh filename=package://nias_description/meshes/RH8D/phalanx_refac.stl scale=0.001 0.001 0.001; visual mesh filename=package://nias_description/meshes/RH8D/phalanx_refac.stl scale=0.001 0.001 0.001
- link r_Rtip: geometry collision mesh filename=package://nias_description/meshes/RH8D/high_res/tip_refac.s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 scale=0.001 0.001 0.001; visual mesh filename=package://nias_description/meshes/RH8D/high_res/tip_refac.s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 scale=0.001 0.001 0.001
- link r_Tbumper: geometry collision mesh filename=package://nias_description/meshes/RH8D/high_res/sensor_refa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 scale=0.001 0.001 0.001; visual mesh filename=package://nias_description/meshes/RH8D/high_res/sensor_refa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 scale=0.001 0.001 0.001
- link r_Tmiddle: geometry collision mesh filename=package://nias_description/meshes/RH8D/thumb_phalanx_refac.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 scale=0.001 0.001 0.001; visual mesh filename=package://nias_description/meshes/RH8D/thumb_phalanx_refac.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 scale=0.001 0.001 0.001
- link r_Tproximal: geometry collision mesh filename=package://nias_description/meshes/RH8D/thumb_phalanx_col.stl scale=0.001 0.001 0.001; visual mesh filename=package://nias_description/meshes/RH8D/thumb_phalanx_refac.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 scale=0.001 0.001 0.001
- link r_Ttip: geometry collision mesh filename=package://nias_description/meshes/RH8D/high_res/tip_refac.s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 scale=0.001 0.001 0.001; visual mesh filename=package://nias_description/meshes/RH8D/high_res/tip_refac.s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 scale=0.001 0.001 0.001
- link r_forearm: geometry collision mesh filename=package://nias_description/meshes/RH8D/forearm_refac.stl scale=0.001 0.001 0.001; visual mesh filename=package://nias_description/meshes/RH8D/forearm_refac.stl scale=0.001 0.001 0.001
- link r_link1: geometry collision box size=0.055 0.055 0.13; visual mesh filename=package://nias_description/meshes/open_manipulator/link_1_r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 scale=0.001 0.001 0.001
- link r_link2: geometry collision box size=0.055 0.1325 0.055; visual mesh filename=package://nias_description/meshes/open_manipulator/link_2_r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 scale=0.001 0.001 0.001
- link r_link3: geometry collision mesh filename=package://nias_description/meshes/open_manipulator/link_3_r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 scale=0.001 0.001 0.001; visual mesh filename=package://nias_description/meshes/open_manipulator/link_3_r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 scale=0.001 0.001 0.001
- link r_link4: geometry collision mesh filename=package://nias_description/meshes/open_manipulator/link_4_r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 scale=0.001 0.001 0.001; visual mesh filename=package://nias_description/meshes/open_manipulator/link_4_r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 scale=0.001 0.001 0.001
- link r_link5: geometry collision box size=0.047 0.08 0.05; visual mesh filename=package://nias_description/meshes/open_manipulator/link_5_r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 scale=0.001 0.001 0.001
- link r_link6: geometry collision mesh filename=package://nias_description/meshes/open_manipulator/link_6_r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 scale=0.001 0.001 0.001; visual mesh filename=package://nias_description/meshes/open_manipulator/link_6_r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 scale=0.001 0.001 0.001
- link r_palm: geometry collision mesh filename=package://nias_description/meshes/RH8D/high_res/right_palm_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 scale=0.001 0.001 0.001; visual mesh filename=package://nias_description/meshes/RH8D/high_res/right_palm_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 scale=0.001 0.001 0.001
- link r_palm_axis: geometry collision mesh filename=package://nias_description/meshes/RH8D/palm_axis_refac.stl scale=0.001 0.001 0.001; visual mesh filename=package://nias_description/meshes/RH8D/palm_axis_refac.stl scale=0.001 0.001 0.001
- link r_thumb_base: geometry collision box size=0 0 0; visual mesh filename=package://nias_description/meshes/RH8D/thumb_base_refac.stl scale=0.001 0.001 0.001
- link right_eye_link: geometry collision box size=0 0 0; visual mesh filename=package://nias_description/meshes/head/BF10M10526S132C_cent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 scale=0.001 0.001 0.001
- link tilt_link: geometry collision box size=0.04 0.042 0.08; visual mesh filename=package://nias_description/meshes/head/tilt_asmbly.stl scale=0.001 0.001 0.001
Joints:
- joint joint_head_tool0: origin xyz=0.0 0.0 0.0975 rpy=0 0 0 -> xyz=0.0 0.0 0.100 rpy=0 0 0
- joint joint_head_tool1: origin xyz=0.224 0.0 0.0975 rpy=0 0 0 -> xyz=0.22 0.0 0.100 rpy=0 0 0
- joint joint_head_y: axis 0 -1 0 -> 0 1 0; limit lower=-3.141592653589793 upper=3.141592653589793 effort=30 velocity=1.0 -> lower=-0.583 upper=1.282 effort=44.7 velocity=6.5; origin xyz=0.0085 0 0.061 rpy=0 0 0 -> xyz=0.007 0 0.0605 rpy=0 0 0
- joint joint_head_z: limit lower=-3.141592653589793 upper=3.141592653589793 effort=30 velocity=1.0 -> lower=-1.5707963267948966 upper=1.5707963267948966 effort=120 velocity=20; origin xyz=0.190 0 0.138 rpy=0 0 0 -> xyz=0.187 -0.001 0.1415 rpy=0 0 0
- joint joint_left_eye: origin xyz=0.1085 0.0466 0.100 rpy=0 0 0 -> xyz=0.111 0.0465 0.0985 rpy=0 0 0
- joint joint_occiput: origin xyz=-0.008 0 0.0325 rpy=0 0 0 -> xyz=0 0 0.032 rpy=0 0 0
- joint joint_right_eye: origin xyz=0.1085 -0.0466 0.100 rpy=0 0 0 -> xyz=0.111 -0.0465 0.0985 rpy=0 0 0
- joint l_joint1: limit lower=-3.141592653589793 upper=0 effort=1000 velocity=6.5 -> lower=-2.5 upper=0 effort=1000 velocity=6.5
- joint l_joint4: limit lower=-3.141592653589793 upper=3.141592653589793 effort=1000 velocity=6.5 -> lower=-2.9 upper=2.9 effort=1000 velocity=6.5
- joint l_joint7: axis 0 0 -1 -> 0 0 1; limit lower=-0.7853981633974483 upper=0.7853981633974483 effort=0.5 velocity=1.0 -> lower=-0.7853981633974483 upper=0.7853981633974483 effort=50 velocity=10.0
- joint l_joint8: limit lower=-0.7853981633974483 upper=0.7853981633974483 effort=0.5 velocity=1.0 -> lower=-0.7853981633974483 upper=0.7853981633974483 effort=50 velocity=10.0
- joint l_jointI1: limit lower=0.0 upper=1.5707963267948966 effort=0.5 velocity=1.0 -> lower=0.0 upper=1.5707963267948966 effort=50 velocity=10.0
- joint l_jointI2: limit lower=0.0 upper=1.5707963267948966 effort=0.5 velocity=1.0 -> lower=0.0 upper=1.5707963267948966 effort=50 velocity=10.0
- joint l_jointI3: limit lower=0.0 upper=1.5707963267948966 effort=0.5 velocity=1.0 -> lower=0.0 upper=1.5707963267948966 effort=50 velocity=10.0
- joint l_jointL1: limit lower=0.0 upper=1.5707963267948966 effort=0.5 velocity=1.0 -> lower=0.0 upper=1.5707963267948966 effort=50 velocity=10.0
- joint l_jointL2: limit lower=0.0 upper=1.5707963267948966 effort=0.5 velocity=1.0 -> lower=0.0 upper=1.5707963267948966 effort=50 velocity=10.0
- joint l_jointL3: limit lower=0.0 upper=1.5707963267948966 effort=0.5 velocity=1.0 -> lower=0.0 upper=1.5707963267948966 effort=50 velocity=10.0
- joint l_jointM1: limit lower=0.0 upper=1.5707963267948966 effort=0.5 velocity=1.0 -> lower=0.0 upper=1.5707963267948966 effort=50 velocity=10.0
- joint l_jointM2: limit lower=0.0 upper=1.5707963267948966 effort=0.5 velocity=1.0 -> lower=0.0 upper=1.5707963267948966 effort=50 velocity=10.0
- joint l_jointM3: limit lower=0.0 upper=1.5707963267948966 effort=0.5 velocity=1.0 -> lower=0.0 upper=1.5707963267948966 effort=50 velocity=10.0
- joint l_jointR1: limit lower=0.0 upper=1.5707963267948966 effort=0.5 velocity=1.0 -> lower=0.0 upper=1.5707963267948966 effort=50 velocity=10.0
- joint l_jointR2: limit lower=0.0 upper=1.5707963267948966 effort=0.5 velocity=1.0 -> lower=0.0 upper=1.5707963267948966 effort=50 velocity=10.0
- joint l_jointR3: limit lower=0.0 upper=1.5707963267948966 effort=0.5 velocity=1.0 -> lower=0.0 upper=1.5707963267948966 effort=50 velocity=10.0
- joint l_jointT0: limit lower=0.0 upper=1.5707963267948966 effort=0.5 velocity=1.0 -> lower=0.0 upper=1.5707963267948966 effort=50 velocity=10.0
- joint l_jointT1: limit lower=0.0 upper=1.5707963267948966 effort=0.5 velocity=1.0 -> lower=0.0 upper=1.5707963267948966 effort=50 velocity=10.0
- joint l_jointT2: limit lower=0.0 upper=1.5707963267948966 effort=0.5 velocity=1.0 -> lower=0.0 upper=1.5707963267948966 effort=50 velocity=10.0
- joint l_jointT3: limit lower=0.0 upper=1.5707963267948966 effort=0.5 velocity=1.0 -> lower=0.0 upper=1.5707963267948966 effort=50 velocity=10.0
- joint r_joint7: limit lower=-0.7853981633974483 upper=0.7853981633974483 effort=0.5 velocity=1.0 -> lower=-0.7853981633974483 upper=0.7853981633974483 effort=50 velocity=10.0
- joint r_joint8: limit lower=-0.7853981633974483 upper=0.7853981633974483 effort=0.5 velocity=1.0 -> lower=-0.7853981633974483 upper=0.7853981633974483 effort=50 velocity=10.0
- joint r_jointI1: limit lower=0.0 upper=1.5707963267948966 effort=0.5 velocity=1.0 -> lower=0.0 upper=1.5707963267948966 effort=50 velocity=10.0
- joint r_jointI2: limit lower=0.0 upper=1.5707963267948966 effort=0.5 velocity=1.0 -> lower=0.0 upper=1.5707963267948966 effort=50 velocity=10.0
- joint r_jointI3: limit lower=0.0 upper=1.5707963267948966 effort=0.5 velocity=1.0 -> lower=0.0 upper=1.5707963267948966 effort=50 velocity=10.0
- joint r_jointL1: limit lower=0.0 upper=1.5707963267948966 effort=0.5 velocity=1.0 -> lower=0.0 upper=1.5707963267948966 effort=50 velocity=10.0
- joint r_jointL2: limit lower=0.0 upper=1.5707963267948966 effort=0.5 velocity=1.0 -> lower=0.0 upper=1.5707963267948966 effort=50 velocity=10.0
- joint r_jointL3: limit lower=0.0 upper=1.5707963267948966 effort=0.5 velocity=1.0 -> lower=0.0 upper=1.5707963267948966 effort=50 velocity=10.0
- joint r_jointM1: limit lower=0.0 upper=1.5707963267948966 effort=0.5 velocity=1.0 -> lower=0.0 upper=1.5707963267948966 effort=50 velocity=10.0
- joint r_jointM2: limit lower=0.0 upper=1.5707963267948966 effort=0.5 velocity=1.0 -> lower=0.0 upper=1.5707963267948966 effort=50 velocity=10.0
- joint r_jointM3: limit lower=0.0 upper=1.5707963267948966 effort=0.5 velocity=1.0 -> lower=0.0 upper=1.5707963267948966 effort=50 velocity=10.0
- joint r_jointR1: limit lower=0.0 upper=1.5707963267948966 effort=0.5 velocity=1.0 -> lower=0.0 upper=1.5707963267948966 effort=50 velocity=10.0
- joint r_jointR2: limit lower=0.0 upper=1.5707963267948966 effort=0.5 velocity=1.0 -> lower=0.0 upper=1.5707963267948966 effort=50 velocity=10.0
- joint r_jointR3: limit lower=0.0 upper=1.5707963267948966 effort=0.5 velocity=1.0 -> lower=0.0 upper=1.5707963267948966 effort=50 velocity=10.0
- joint r_jointT0: limit lower=0.0 upper=1.5707963267948966 effort=0.5 velocity=1.0 -> lower=0.0 upper=1.5707963267948966 effort=50 velocity=10.0
- joint r_jointT1: limit lower=0.0 upper=1.5707963267948966 effort=0.5 velocity=1.0 -> lower=0.0 upper=1.5707963267948966 effort=50 velocity=10.0
- joint r_jointT2: limit lower=0.0 upper=1.5707963267948966 effort=0.5 velocity=1.0 -> lower=0.0 upper=1.5707963267948966 effort=50 velocity=10.0
- joint r_jointT3: limit lower=0.0 upper=1.5707963267948966 effort=0.5 velocity=1.0 -> lower=0.0 upper=1.5707963267948966 effort=50 velocity=10.0
